Commit message: switched to waffle

File: turtlebot3_description/urdf/turtlebot3_waffle.urdf (robot description, URDF)
Before this commit: robot turtlebot3_waffle, 13 links, 12 joints
Links:
- removed link ${namespace}base_footprint
- removed link ${namespace}base_link
- removed link ${namespace}base_scan
- removed link ${namespace}camera_depth_frame
- removed link ${namespace}camera_depth_optical_frame
- removed link ${namespace}camera_link
- removed link ${namespace}camera_rgb_frame
- removed link ${namespace}camera_rgb_optical_frame
- removed link ${namespace}caster_back_left_link
- removed link ${namespace}caster_back_right_link
- removed link ${namespace}imu_link
- removed link ${namespace}wheel_left_link
- removed link ${namespace}wheel_right_link
- added link turtlebotbase_footprint
- added link turtlebotbase_link, mass 1.3729096e+00; collision box size=0.266 0.266 0.094; visual mesh filename=../meshes/bases/waffle_base.stl scale=0.001 0.001 0.001
- added link turtlebotbase_scan, mass 0.114; collision cylinder length=0.0315 radius=0.055; visual mesh filename=../meshes/sensors/lds.stl scale=0.001 0.001 0.001
- added link turtlebotcamera_depth_frame
- added link turtlebotcamera_depth_optical_frame
- added link turtlebotcamera_link; collision box size=0.012 0.132 0.020; visual mesh filename=../meshes/sensors/r200.dae scale=0.001 0.001 0.001
- added link turtlebotcamera_rgb_frame
- added link turtlebotcamera_rgb_optical_frame
- added link turtlebotcaster_back_left_link, mass 0.005; collision box size=0.030 0.009 0.020
- added link turtlebotcaster_back_right_link, mass 0.005; collision box size=0.030 0.009 0.020
- added link turtlebotimu_link
- added link turtlebotwheel_left_link, mass 2.8498940e-02; collision cylinder length=0.018 radius=0.033; visual mesh filename=../meshes/wheels/left_tire.stl scale=0.001 0.001 0.001
- added link turtlebotwheel_right_link, mass 2.8498940e-02; collision cylinder length=0.018 radius=0.033; visual mesh filename=../meshes/wheels/right_tire.stl scale=0.001 0.001 0.001
Joints:
- removed joint ${namespace}base_joint
- removed joint ${namespace}camera_depth_joint
- removed joint ${namespace}camera_depth_optical_joint
- removed joint ${namespace}camera_joint
- removed joint ${namespace}camera_rgb_joint
- removed joint ${namespace}camera_rgb_optical_joint
- removed joint ${namespace}caster_back_left_joint
- removed joint ${namespace}caster_back_right_joint
- removed joint ${namespace}imu_joint
- removed joint ${namespace}scan_joint
- removed joint ${namespace}wheel_left_joint
- removed joint ${namespace}wheel_right_joint
- added joint turtlebotbase_joint: type fixed, parent turtlebotbase_footprint, child turtlebotbase_link, origin xyz=0 0 0.010 rpy=0 0 0
- added joint turtlebotcamera_depth_joint: type fixed, parent turtlebotcamera_link, child turtlebotcamera_depth_frame, origin xyz=0.005 0.028 0.013 rpy=0 0 0
- added joint turtlebotcamera_depth_optical_joint: type fixed, parent turtlebotcamera_depth_frame, child turtlebotcamera_depth_optical_frame, origin xyz=0 0 0 rpy=-1.57 0 -1.57
- added joint turtlebotcamera_joint: type fixed, parent turtlebotbase_link, child turtlebotcamera_link, origin xyz=0.064 -0.065 0.094 rpy=0 0 0
- added joint turtlebotcamera_rgb_joint: type fixed, parent turtlebotcamera_link, child turtlebotcamera_rgb_frame, origin xyz=0.005 0.018 0.013 rpy=0 0 0
- added joint turtlebotcamera_rgb_optical_joint: type fixed, parent turtlebotcamera_rgb_frame, child turtlebotcamera_rgb_optical_frame, origin xyz=0 0 0 rpy=-1.57 0 -1.57
- added joint turtlebotcaster_back_left_joint: type fixed, parent turtlebotbase_link, child turtlebotcaster_back_left_link, origin xyz=-0.177 0.064 -0.004 rpy=-1.57 0 0
- added joint turtlebotcaster_back_right_joint: type fixed, parent turtlebotbase_link, child turtlebotcaster_back_right_link, origin xyz=-0.177 -0.064 -0.004 rpy=-1.57 0 0
- added joint turtlebotimu_joint: type fixed, parent turtlebotbase_link, child turtlebotimu_link, origin xyz=0.0 0 0.068 rpy=0 0 0
- added joint turtlebotscan_joint: type fixed, parent turtlebotbase_link, child turtlebotbase_scan, origin xyz=-0.064 0 0.122 rpy=0 0 0
- added joint turtlebotwheel_left_joint: type continuous, parent turtlebotbase_link, child turtlebotwheel_left_link, origin xyz=0.0 0.144 0.023 rpy=-1.57 0 0, axis 0 0 1
- added joint turtlebotwheel_right_joint: type continuous, parent turtlebotbase_link, child turtlebotwheel_right_link, origin xyz=0.0 -0.144 0.023 rpy=-1.57 0 0, axis 0 0 1

Commit message: tf tree added

File: turtlebot3_description/urdf/turtlebot3_waffle.urdf (robot description, URDF)
Before this commit: robot turtlebot3_waffle, 13 links, 12 joints
Links:
- removed link turtlebotbase_footprint
- removed link turtlebotbase_link
- removed link turtlebotbase_scan
- removed link turtlebotcamera_depth_frame
- removed link turtlebotcamera_depth_optical_frame
- removed link turtlebotcamera_link
- removed link turtlebotcamera_rgb_frame
- removed link turtlebotcamera_rgb_optical_frame
- removed link turtlebotcaster_back_left_link
- removed link turtlebotcaster_back_right_link
- removed link turtlebotimu_link
- removed link turtlebotwheel_left_link
- removed link turtlebotwheel_right_link
- added link base_footprint
- added link base_link, mass 1.3729096e+00; collision box size=0.266 0.266 0.094; visual mesh filename=../meshes/bases/waffle_base.stl scale=0.001 0.001 0.001
- added link base_scan, mass 0.114; collision cylinder length=0.0315 radius=0.055; visual mesh filename=../meshes/sensors/lds.stl scale=0.001 0.001 0.001
- added link camera_depth_frame
- added link camera_depth_optical_frame
- added link camera_link; collision box size=0.012 0.132 0.020; visual mesh filename=../meshes/sensors/r200.dae scale=0.001 0.001 0.001
- added link camera_rgb_frame
- added link camera_rgb_optical_frame
- added link caster_back_left_link, mass 0.005; collision box size=0.030 0.009 0.020
- added link caster_back_right_link, mass 0.005; collision box size=0.030 0.009 0.020
- added link imu_link
- added link wheel_left_link, mass 2.8498940e-02; collision cylinder length=0.018 radius=0.033; visual mesh filename=../meshes/wheels/left_tire.stl scale=0.001 0.001 0.001
- added link wheel_right_link, mass 2.8498940e-02; collision cylinder length=0.018 radius=0.033; visual mesh filename=../meshes/wheels/right_tire.stl scale=0.001 0.001 0.001
Joints:
- removed joint turtlebotbase_joint
- removed joint turtlebotcamera_depth_joint
- removed joint turtlebotcamera_depth_optical_joint
- removed joint turtlebotcamera_joint
- removed joint turtlebotcamera_rgb_joint
- removed joint turtlebotcamera_rgb_optical_joint
- removed joint turtlebotcaster_back_left_joint
- removed joint turtlebotcaster_back_right_joint
- removed joint turtlebotimu_joint
- removed joint turtlebotscan_joint
- removed joint turtlebotwheel_left_joint
- removed joint turtlebotwheel_right_joint
- added joint base_joint: type fixed, parent base_footprint, child base_link, origin xyz=0 0 0.010 rpy=0 0 0
- added joint camera_depth_joint: type fixed, parent camera_link, child camera_depth_frame, origin xyz=0.005 0.028 0.013 rpy=0 0 0
- added joint camera_depth_optical_joint: type fixed, parent camera_depth_frame, child camera_depth_optical_frame, origin xyz=0 0 0 rpy=-1.57 0 -1.57
- added joint camera_joint: type fixed, parent base_link, child camera_link, origin xyz=0.064 -0.065 0.094 rpy=0 0 0
- added joint camera_rgb_joint: type fixed, parent camera_link, child camera_rgb_frame, origin xyz=0.005 0.018 0.013 rpy=0 0 0
- added joint camera_rgb_optical_joint: type fixed, parent camera_rgb_frame, child camera_rgb_optical_frame, origin xyz=0 0 0 rpy=-1.57 0 -1.57
- added joint caster_back_left_joint: type fixed, parent base_link, child caster_back_left_link, origin xyz=-0.177 0.064 -0.004 rpy=-1.57 0 0
- added joint caster_back_right_joint: type fixed, parent base_link, child caster_back_right_link, origin xyz=-0.177 -0.064 -0.004 rpy=-1.57 0 0
- added joint imu_joint: type fixed, parent base_link, child imu_link, origin xyz=0.0 0 0.068 rpy=0 0 0
- added joint scan_joint: type fixed, parent base_link, child base_scan, origin xyz=-0.064 0 0.122 rpy=0 0 0
- added joint wheel_left_joint: type continuous, parent base_link, child wheel_left_link, origin xyz=0.0 0.144 0.023 rpy=-1.57 0 0, axis 0 0 1
- added joint wheel_right_joint: type continuous, parent base_link, child wheel_right_link, origin xyz=0.0 -0.144 0.023 rpy=-1.57 0 0, axis 0 0 1
